File: Output Indicators.kicad_sch (KiCad schematic)
At the start: 76 parts, among them U201 1G126, U202 1G126, U203 74HC595, U204 1G126, U205 1G126, U206 74HC595, U207 1G126, U208 1G126, U209 1G126, U210 1G126, U211 74HC595, U212 74HC595, U213 1G126, U214 1G126, U215 1G126, U216 1G126, U217 1G126, U218 1G126, U219 1G126, U220 1G126

Commit message: First version of layout
Parts:
- added D217, D218: MXA8-PW40-0000, 0_NRD_footprints:LED_Luxeon3535_3.5x3.7mm, symbol 00_projectlib:LED_LUML_MXA8-PW40-0000
- added J201: BM05B, 0_NRD_footprints:J_BM05B-GHS-TBT, symbol 0_NRD_Connectors:CON_JST_BM05B-GHS-TBT
- added R217, R218: 39R, Resistor_SMD:R_0805_2012Metric, symbol 0_NRD_Resistors:R_0805.__39R
- added U220, U221: 1G126, Package_TO_SOT_SMD:SOT-353_SC-70-5, symbol 0_NRD_Level_and_logic:LOG_7400_1G126
- renumbered C204 to C201, C203 to C202, C202 to C203, C201 to C204, D211 to D202, D215 to D203, D217 to D204, D219 to D205, D221 to D206, D223 to D207, D225 to D208, D202 to D209, D212 to D210, D216 to D211, D218 to D212, D220 to D213, D222 to D214, D224 to D215, D226 to D216, D203 to D219, D204 to D220, D205 to D221, D206 to D222, D207 to D223, D208 to D224, D209 to D225, D210 to D226, D213 to D227, D214 to D228, R211 to R202, R215 to R203, R217 to R204, R219 to R205, R221 to R206, R223 to R207, R225 to R208, R202 to R209, R212 to R210, R216 to R211, R218 to R212, R220 to R213, R222 to R214, R224 to R215, R226 to R216, R203 to R219, R204 to R220, R205 to R221, R206 to R222, R207 to R223, R208 to R224, R209 to R225, R210 to R226, R213 to R227, R214 to R228, U211 to U201, U201 to U202, U204 to U203, U207 to U204, U209 to U205, U213 to U206, U215 to U207, U217 to U208, U219 to U209, U212 to U210, U202 to U211, U205 to U212, U208 to U213, U210 to U214, U214 to U215, U218 to U217, U220 to U218, U203 to U219, U206 to U222
Connections:
- net +3.3V: now also J201.1 (Pin_1), U220.5 (VCC), U221.5 (VCC)
- net CLK: now also J201.3 (Pin_3)
- net GND: now also D217.1 (K), D218.1 (K), J201.5 (Pin_5), J201.MP (MountPin), U220.3 (GND), U221.3 (GND)
- net LATCH: now also J201.4 (Pin_4)
- net OE: now also U220.1 (OE), U221.1 (OE)
- net at R222.1: now also U219.5 (QF); no longer U219.3 (QD)
- net at R227.1: now also U222.2 (QC); no longer U222.15 (QA)
- net at R221.1: now also U219.4 (QE); no longer U219.2 (QC)
- net at R223.1: now also U219.6 (QG); no longer U219.4 (QE)
- net at U222.1 (QB): now also R226.1; no longer R228.1
- net at U222.3 (QD): now also R228.1
- net at U222.4 (QE): now also J201.2 (Pin_2)
- net at R224.1: now also U219.7 (QH); no longer U219.5 (QF)
- net at U219.1 (QB): now also U221.2 (A); no longer R220.1
- net at U219.15 (QA): now also U220.2 (A); no longer R219.1
- net at R225.1: now also U222.15 (QA); no longer U219.6 (QG)
- new net: R218.1, U221.4 (Y)
- new net: D218.2 (A), R218.2
- new net: R217.1, U220.4 (Y)
- new net: R220.1, U219.3 (QD)
- new net: R219.1, U219.2 (QC)
- new net: D217.2 (A), R217.2
- no-connect marks 7 -> 4
Other:
- moved on the sheet: C203, C204, D219, D220, D221, D222, D223, D224, D225, D226, D227, D228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

Commit message: Added new version of artifact generator
Parts:
- J201: value BM05B -> BM06B; footprint 0_NRD_footprints:J_BM05B-GHS-TBT -> 0_NRD_footprints:J_BM06B-GHS-TBT; symbol 0_NRD_Connectors:CON_JST_BM05B-GHS-TBT -> 0_NRD_Connectors:CON_JST_BM06B-GHS-TBT; MPN BM05B-GHS-TBT(LF)(SN) -> BM06B-GHS-TBT(LF)(SN); S1 Description Connector Header Surface Mount 5 position 0.049" (1.25mm) -> Connector Header Surface Mount 6 position 0.049" (1.25mm); S1 Part link https://mou.sr/4rhQYiT -> https://mou.sr/43ABJaA; S1 Part number 306-BM05BGHSTBTLFSN -> 306-BM06BGHSTBTLFSN; S1 Price @ 100 0.242 -> 0.288
Connections:
- net +3.3V: now also J201.2 (Pin_2); no longer J201.1 (Pin_1)
- net CLK: now also J201.4 (Pin_4); no longer J201.3 (Pin_3)
- net GND: now also J201.6 (Pin_6); no longer J201.5 (Pin_5)
- net LATCH: now also J201.5 (Pin_5); no longer J201.4 (Pin_4)
- net at U222.4 (QE): now also J201.3 (Pin_3); no longer J201.2 (Pin_2)
- new net VBUS: J201.1 (Pin_1)
Changed lines of the file:
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@@
 	(wire
 		(pts
-			(xy 308.61 121.92) (xy 309.88 121.92)
+			(xy 306.07 121.92) (xy 309.88 121.92)
 		)
 		(stroke
@@
 	(wire
 		(pts
-			(xy 308.61 120.65) (xy 308.61 121.92)
+			(xy 306.07 120.65) (xy 306.07 121.92)
 		)
 		(stroke
@@
 	)
 	(symbol
+		(lib_id "power:VBUS")
+		(at 309.88 119.38 0)
+		(unit 1)
+		(exclude_from_sim no)
+		(in_bom yes)
+		(on_board yes)
+		(dnp no)
+		(property "Reference" "#PWR0275"
+			(at 309.88 123.19 0)
+			(effects
+				(font
+					(size 1.27 1.27)
+				)
+				(hide yes)
+			)
+		)
+		(property "Value" "VBUS"
+			(at 309.88 115.316 0)
+			(effects
+				(font
+					(size 1.27 1.27)
+				)
+			)
+		)
+		(property "Footprint" ""
+			(at 309.88 119.38 0)
+			(effects
+				(font
+					(size 1.27 1.27)
+				)
+				(hide yes)
+			)
+		)
+		(property "Datasheet" ""
+			(at 309.88 119.38 0)
+			(effects
+				(font
+					(size 1.27 1.27)
+				)
+				(hide yes)
+			)
+		)
+		(property "Description" "Power symbol creates a global label with name \"VBUS\""
+			(at 309.88 119.38 0)
+			(effects
+				(font
+					(size 1.27 1.27)
+				)
+				(hide yes)
+			)
+		)
+		(pin "1"
+		)
+		(instances
+			(project "2026-NURDspace-PPS"
+				(path "/1b1d42dc-f63c-49d9-9b61-b09c30b6ea01/e958a2e9-b753-4874-981c-670674a7fa9b"
+					(reference "#PWR0275")
+					(unit 1)
+				)
+			)
+		)
+	)
+	(symbol
 		(lib_id "00_projectlib:LED_LUML_MXA8-PW40-0000")
 		(at 190.5 194.31 90)
@@
 	)
 	(symbol
-		(lib_id "0_NRD_Connectors:CON_JST_BM05B-GHS-TBT")
-		(at 314.96 127 0)
+		(lib_id "0_NRD_Connectors:CON_JST_BM06B-GHS-TBT")
+		(at 314.96 125.73 0)
 		(unit 1)
 		(exclude_from_sim no)
@@
 		(fields_autoplaced yes)
 		(property "Reference" "J201"
-			(at 317.5 126.0855 0)
+			(at 317.5 124.8155 0)
 			(effects
 				(font
@@
 			)
 		)
-		(property "Value" "BM05B"
-			(at 317.5 128.6255 0)
+		(property "Value" "BM06B"
+			(at 317.5 127.3555 0)
 			(effects
 				(font
@@
 			)
 		)
-		(property "Footprint" "0_NRD_footprints:J_BM05B-GHS-TBT"
-			(at 316.484 93.98 0)
+		(property "Footprint" "0_NRD_footprints:J_BM06B-GHS-TBT"
+			(at 316.484 92.71 0)
 			(effects
 				(font
@@
 		)
 		(property "Datasheet" "https://www.jst-mfg.com/product/pdf/eng/eGH.pdf"
-			(at 321.564 93.98 0)
+			(at 321.564 92.71 0)
 			(effects
 				(font
@@
 			)
 		)
-		(property "Description" "Connector Header Surface Mount 5 position 0.049\" (1.25mm)"
-			(at 320.548 94.234 0)
+		(property "Description" "Connector Header Surface Mount 6 position 0.049\" (1.25mm)"
+			(at 320.548 92.964 0)
 			(effects
 				(font
@@
 			)
 		)
-		(property "S1 Price @ 100" "0.242"
-			(at 314.452 94.234 0)
+		(property "S1 Price @ 100" "0.288"
+			(at 314.452 92.964 0)
 			(effects
 				(font
@@
 			)
 		)
-		(property "S1 Description" "Connector Header Surface Mount 5 position 0.049\" (1.25mm)"
-			(at 321.564 93.98 0)
+		(property "S1 Description" "Connector Header Surface Mount 6 position 0.049\" (1.25mm)"
+			(at 321.564 92.71 0)
 			(effects
 				(font
@@
 			)
 		)
-		(property "S1 Part number" "306-BM05BGHSTBTLFSN"
-			(at 321.564 93.98 0)
+		(property "S1 Part number" "306-BM06BGHSTBTLFSN"
+			(at 321.564 92.71 0)
 			(effects
 				(font
@@
 			)
 		)
-		(property "S1 Part link" "https://mou.sr/4rhQYiT"
-			(at 321.564 93.98 0)
+		(property "S1 Part link" "https://mou.sr/43ABJaA"
+			(at 321.564 92.71 0)
 			(effects
 				(font
@@
 			)
 		)
-		(property "MPN" "BM05B-GHS-TBT(LF)(SN) "
-			(at 317.754 94.742 0)
+		(property "MPN" "BM06B-GHS-TBT(LF)(SN) "
+			(at 317.754 93.472 0)
 			(effects
 				(font
@@
 		)
 		(property "MF" "JST"
-			(at 316.23 38.1 0)
+			(at 316.23 36.83 0)
 			(effects
 				(font
@@
 		(pin "MP"
 		)
+		(pin "6"
+		)
 		(instances
 			(project ""
@@
 	(symbol
 		(lib_id "power:+3.3V")
-		(at 308.61 120.65 0)
+		(at 306.07 120.65 0)
 		(unit 1)
 		(exclude_from_sim no)
@@
 		(dnp no)
 		(property "Reference" "#PWR0272"
-			(at 308.61 124.46 0)
+			(at 306.07 124.46 0)
 			(effects
 				(font
@@
 		)
 		(property "Value" "+3.3V"
-			(at 308.61 116.586 0)
+			(at 306.07 116.586 0)
 			(effects
 				(font
@@
 		)
 		(property "Footprint" ""
-			(at 308.61 120.65 0)
+			(at 306.07 120.65 0)
 			(effects
 				(font
@@
 		)
 		(property "Datasheet" ""
-			(at 308.61 120.65 0)
+			(at 306.07 120.65 0)
 			(effects
 				(font
@@
 		)
 		(property "Description" "Power symbol creates a global label with name \"+3.3V\""
-			(at 308.61 120.65 0)
+			(at 306.07 120.65 0)
 			(effects
 				(font
